Commit message: add tool link

File: src/urdfs/ur3/ur_macro.xacro (robot description, xacro)
@@ -313,5 +313,5 @@
         <origin xyz="0 0 0.01" rpy="0 0 0"/>
         <geometry>
-          <cylinder length="0.02" radius="0.03"/>
+          <cylinder length="0.02" radius="0.04"/>
         </geometry>
       </visual>
@@ -319,5 +319,5 @@
         <origin xyz="0 0 0.01" rpy="0 0 0"/>
         <geometry>
-          <cylinder length="0.02" radius="0.03"/>
+          <cylinder length="0.02" radius="0.04"/>
         </geometry>
       </collision>
